File: Kicad_Nemo75/Kicad_Nemo75.kicad_sch (KiCad schematic)
At the start: 206 parts, among them J1 Conn_01x08_Pin, J2 USB_A, J4 USB_A, J5 USB_A, J6 USB_A, J7 USB_B_Micro, SW1 SW_Push, SW10 SW_Push, SW11 SW_Push, SW12 SW_Push, SW13 SW_Push, SW14 SW_Push, SW15 RotaryEncoder_Switch, SW16 RotaryEncoder_Switch, SW17 SW_Push, SW18 SW_Push, SW19 SW_Push, SW2 SW_Push, SW20 SW_Push, SW21 SW_Push, SW22 SW_Push, SW23 SW_Push, SW24 SW_Push, SW25 SW_Push, SW26 SW_Push, SW27 SW_Push, SW28 SW_Push, SW29 SW_Push, SW3 SW_Push, SW30 SW_Push, SW31 SW_Push, SW32 SW_Push, SW33 SW_Push, SW34 SW_Push, SW35 SW_Push, SW36 SW_Push, SW37 SW_Push, SW38 SW_Push, SW39 SW_Push, SW4 SW_Push, SW40 SW_Push, SW41 SW_Push, SW42 SW_Push, SW43 SW_Push, SW44 SW_Push, SW45 SW_Push, SW46 SW_Push, SW47 SW_Push, SW48 SW_Push, SW49 SW_Push, SW5 SW_Push, SW50 SW_Push, SW51 SW_Push, SW52 SW_Push, SW53 SW_Push, SW54 SW_Push, SW55 SW_Push, SW56 SW_Push, SW57 SW_Push, SW58 SW_Push, SW59 SW_Push, SW6 SW_Push, SW60 SW_Push, SW61 SW_Push, SW62 SW_Push, SW63 SW_Push, SW64 SW_Push, SW65 SW_Push, SW66 SW_Push, SW67 SW_Push, SW68 SW_Push, SW69 SW_Push, SW7 SW_Push, SW70 SW_Push, SW71 SW_Push, SW72 SW_Push, SW73 SW_Push, SW74 SW_Push, SW75 SW_Push, SW76 SW_Push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

Commit message: schematic completed with stabilizers and a friki DUPLEX MATRIX yeh the japanese one
Parts:
- added S1: MX_stab, PCM_marbastlib-mx:STAB_MX_P_6.25u, symbol PCM_marbastlib-mx:MX_stab
- added S2, S3: MX_stab, PCM_marbastlib-mx:STAB_MX_P_2.75u, symbol PCM_marbastlib-mx:MX_stab
- added S4: MX_stab, PCM_marbastlib-mx:STAB_MX_P_2u, symbol PCM_marbastlib-mx:MX_stab
- added S5: MX_stab, PCM_marbastlib-mx:STAB_MX_P_2.25u, symbol PCM_marbastlib-mx:MX_stab
- C1, C2, C3, C4, C5, C6, C7: footprint (none) -> Capacitor_SMD:C_1206_3216Metric_Pad1.33x1.80mm_HandSolder
- D1, D10, D107, D11, D12, D13, D14, D15, D16, D17, D18, D19, D2, D20, D21, D22, D23, D24, D25, D26, D27, D28, D29, D3, D30, D31, D32, D33, D34, D35, D36, D37, D38, D39, D4, D40, D41, D42, D43, D44, D45, D46, D47, D48, D49, D5, D50, D51, D52, D53, D54, D55, D56, D57, D58, D59, D6, D60, D61, D62, D63, D64, D65, D66, D67, D68, D69, D7, D70, D71, D72, D73, D74, D75, D76, D77, D78, D79, D8, D80, D81, D82, D83, D84, D9: footprint Diode_THT:D_DO-41_SOD81_P10.16mm_Horizontal -> Diode_THT:D_DO-35_SOD27_P7.62mm_Horizontal
- J2, J4, J5, J6: footprint LED_SMD:LED_SK6812_PLCC4_5.0x5.0mm_P3.2mm -> Connector_USB:USB_A_Molex_67643_Horizontal
- J7: footprint (none) -> Connector_USB:USB_Micro-B_Wuerth_629105150521
- SW1, SW10, SW11, SW12, SW13, SW14, SW17, SW18, SW19, SW2, SW20, SW21, SW22, SW23, SW24, SW25, SW26, SW27, SW28, SW29, SW3, SW30, SW31, SW32, SW33, SW34, SW35, SW36, SW37, SW38, SW39, SW4, SW40, SW41, SW42, SW43, SW44, SW45, SW46, SW47, SW48, SW49, SW5, SW50, SW51, SW52, SW53, SW54, SW55, SW56, SW57, SW58, SW59, SW6, SW60, SW61, SW62, SW63, SW64, SW65, SW66, SW67, SW68, SW69, SW7, SW70, SW71, SW72, SW73, SW74, SW75, SW76, SW77, SW78, SW79, SW8, SW80, SW81, SW82, SW83, SW84, SW9: footprint Button_Switch_SMD:Nidec_Copal_CAS-120A -> PCM_marbastlib-mx:SW_MX_HS_CPG151101S11_1u
- SW15, SW16: footprint (none) -> Rotary_Encoder:RotaryEncoder_Alps_EC11E-Switch_Vertical_H20mm
Connections:
- net +3.3V: now also D100.3 (VDD), D101.3 (VDD), D102.3 (VDD), D103.3 (VDD), D104.3 (VDD), D105.3 (VDD), D106.3 (VDD), D96.3 (VDD), D97.3 (VDD), D98.3 (VDD), D99.3 (VDD); no longer D100.1 (VSS), D101.1 (VSS), D102.1 (VSS), D103.1 (VSS), D104.1 (VSS), D105.1 (VSS), D106.1 (VSS), D96.1 (VSS), D97.1 (VSS), D98.1 (VSS), D99.1 (VSS)
- net COL 1: now also D1.1 (K), D11.1 (K), D12.2 (A), D2.2 (A), D21.1 (K), D22.2 (A), D31.1 (K), D32.2 (A), D41.1 (K), D42.2 (A), D51.1 (K), D52.2 (A), D61.1 (K), D62.2 (A), D71.1 (K), D72.2 (A), D81.1 (K), D82.2 (A); no longer SW1.2, SW11.2, SW21.2, SW31.2, SW40.2, SW49.2, SW58.2, SW67.2, SW76.2
- net COL 2: now also D13.1 (K), D14.2 (A), D23.1 (K), D24.2 (A), D3.1 (K), D33.1 (K), D34.2 (A), D4.2 (A), D43.1 (K), D44.2 (A), D53.1 (K), D54.2 (A), D63.1 (K), D64.2 (A), D73.1 (K), D74.2 (A), D83.1 (K), D84.2 (A); no longer SW12.2, SW2.2, SW22.2, SW32.2, SW41.2, SW50.2, SW59.2, SW68.2, SW77.2
- net COL 3: now also D15.1 (K), D16.2 (A), D25.1 (K), D26.2 (A), D35.1 (K), D36.2 (A), D45.1 (K), D46.2 (A), D5.1 (K), D55.1 (K), D56.2 (A), D6.2 (A), D65.1 (K), D66.2 (A), D75.1 (K), D76.2 (A); no longer SW13.2, SW23.2, SW3.2, SW33.2, SW42.2, SW51.2, SW60.2, SW69.2, SW78.2
- net COL 4: now also D17.1 (K), D18.2 (A), D27.1 (K), D28.2 (A), D37.1 (K), D38.2 (A), D47.1 (K), D48.2 (A), D57.1 (K), D58.2 (A), D67.1 (K), D68.2 (A), D7.1 (K), D77.1 (K), D78.2 (A), D8.2 (A); no longer SW14.2, SW24.2, SW34.2, SW4.2, SW43.2, SW52.2, SW61.2, SW70.2, SW79.2
- net COL 5: now also D10.2 (A), D19.1 (K), D20.2 (A), D29.1 (K), D30.2 (A), D39.1 (K), D40.2 (A), D49.1 (K), D50.2 (A), D59.1 (K), D60.2 (A), D69.1 (K), D70.2 (A), D79.1 (K), D80.2 (A), D9.1 (K); no longer SW20.2, SW25.2, SW35.2, SW44.2, SW5.2, SW53.2, SW62.2, SW71.2, SW80.2
- net GND: now also D100.1 (VSS), D101.1 (VSS), D102.1 (VSS), D103.1 (VSS), D104.1 (VSS), D105.1 (VSS), D106.1 (VSS), D96.1 (VSS), D97.1 (VSS), D98.1 (VSS), D99.1 (VSS); no longer D100.3 (VDD), D101.3 (VDD), D102.3 (VDD), D103.3 (VDD), D104.3 (VDD), D105.3 (VDD), D106.3 (VDD), D96.3 (VDD), D97.3 (VDD), D98.3 (VDD), D99.3 (VDD)
- net LED: now also A1.26 (GPIO20); no longer A1.31 (GPIO26_ADC0)
- net RE 1 A: now also A1.19 (GPIO14); no longer A1.29 (GPIO22)
- net RE 1 B: now also A1.22 (GPIO17); no longer A1.26 (GPIO20)
- net RE 2 A: now also A1.20 (GPIO15); no longer A1.27 (GPIO21)
- net RE 2 B: now also A1.21 (GPIO16); no longer A1.25 (GPIO19)
- net RE 2 OUT: now also D84.1 (K); no longer D84.2 (A)
- net ROW 1: now also SW1.1, SW10.1, SW2.1, SW3.1, SW4.1, SW5.1, SW6.1, SW7.1, SW8.1, SW9.1; no longer D1.1 (K), D10.1 (K), D2.1 (K), D3.1 (K), D4.1 (K), D5.1 (K), D6.1 (K), D7.1 (K), D8.1 (K), D9.1 (K)
- net ROW 2: now also SW11.1, SW12.1, SW13.1, SW14.1, SW17.1, SW18.1, SW19.1, SW20.1, SW21.1, SW22.1; no longer D11.1 (K), D12.1 (K), D13.1 (K), D14.1 (K), D15.1 (K), D16.1 (K), D17.1 (K), D18.1 (K), D19.1 (K), D84.1 (K)
- net ROW 3: now also SW23.1, SW24.1, SW25.1, SW26.1, SW27.1, SW28.1, SW29.1, SW30.1, SW31.1, SW32.1; no longer D20.1 (K), D21.1 (K), D22.1 (K), D23.1 (K), D24.1 (K), D25.1 (K), D26.1 (K), D27.1 (K), D28.1 (K), D83.1 (K)
- net ROW 4: now also SW33.1, SW34.1, SW35.1, SW36.1, SW37.1, SW38.1, SW39.1, SW40.1, SW41.1, SW42.1; no longer D29.1 (K), D30.1 (K), D31.1 (K), D32.1 (K), D33.1 (K), D34.1 (K), D35.1 (K), D36.1 (K), D37.1 (K)
- net ROW 5: now also SW43.1, SW44.1, SW45.1, SW46.1, SW47.1, SW48.1, SW49.1, SW50.1, SW51.1, SW52.1; no longer D38.1 (K), D39.1 (K), D40.1 (K), D41.1 (K), D42.1 (K), D43.1 (K), D44.1 (K), D45.1 (K), D46.1 (K)
- net ROW 6: now also SW53.1, SW54.1, SW55.1, SW56.1, SW57.1, SW58.1, SW59.1, SW60.1, SW61.1, SW62.1; no longer D47.1 (K), D48.1 (K), D49.1 (K), D50.1 (K), D51.1 (K), D52.1 (K), D53.1 (K), D54.1 (K), D55.1 (K)
- net ROW 7: now also SW63.1, SW64.1, SW65.1, SW66.1, SW67.1, SW68.1, SW69.1, SW70.1, SW71.1, SW72.1; no longer D56.1 (K), D57.1 (K), D58.1 (K), D59.1 (K), D60.1 (K), D61.1 (K), D62.1 (K), D63.1 (K), D64.1 (K)
- net ROW 8: now also SW73.1, SW74.1, SW75.1, SW76.1, SW77.1, SW78.1, SW79.1, SW80.1, SW81.1, SW82.1; no longer D65.1 (K), D66.1 (K), D67.1 (K), D68.1 (K), D69.1 (K), D70.1 (K), D71.1 (K), D72.1 (K), D73.1 (K)
- net SCL: now also A1.24 (GPIO18); no longer A1.32 (GPIO27_ADC1)
- net SDA: now also A1.25 (GPIO19); no longer A1.34 (GPIO28_ADC2)
- net at D39.2 (A): now also SW41.2; no longer SW41.1
- net at D41.2 (A): now also SW43.2; no longer SW43.1
- net at D43.2 (A): now also SW45.2; no longer SW45.1
- net at D35.2 (A): now also SW37.2; no longer SW37.1
- net at D81.2 (A): now also SW83.2; no longer SW83.1
- net at D53.2 (A): now also SW55.2; no longer SW55.1
- net at D51.2 (A): now also SW53.2; no longer SW53.1
- net at D65.2 (A): now also SW67.2; no longer SW67.1
- net at D29.2 (A): now also SW31.2; no longer SW31.1
- net at D11.2 (A): now also SW11.2; no longer SW11.1
- net at D57.2 (A): now also SW59.2; no longer SW59.1
- net at D5.2 (A): now also SW5.2; no longer SW5.1
- net BLK: now reaches J1.BLK
- net BLK: now also A1.32 (GPIO27_ADC1)
- net CS: now reaches J1.CS
- net CS: now also A1.31 (GPIO26_ADC0)
- net DC: now reaches J1.DC
- net DC: now also A1.29 (GPIO22)
- net RES: now reaches J1.RES
- net RES: now also A1.27 (GPIO21)
- net at D79.2 (A): now also SW81.2; no longer SW81.1
- net at D49.2 (A): now also SW51.2; no longer SW51.1
- net at D1.2 (A): now also SW1.2; no longer SW1.1
- net at D37.2 (A): now also SW39.2; no longer SW39.1
- net at D98.2 (DIN): now also D99.4 (DOUT); no longer D97.4 (DOUT)
- net at D98.4 (DOUT): now also D97.2 (DIN); no longer D99.2 (DIN)
- net at D77.2 (A): now also SW79.2; no longer SW79.1
- net at D17.2 (A): now also SW19.2; no longer SW17.1
- net at D100.2 (DIN): now also D101.4 (DOUT); no longer D99.4 (DOUT)
- net at D100.4 (DOUT): now also D99.2 (DIN); no longer D101.2 (DIN)
- net at D59.2 (A): now also SW61.2; no longer SW61.1
- net at D75.2 (A): now also SW77.2; no longer SW77.1
- net at D23.2 (A): now also SW25.2; no longer SW24.1
- net at D69.2 (A): now also SW71.2; no longer SW71.1
- net at D106.2 (DIN): now also D95.4 (DOUT); no longer D105.4 (DOUT)
- net at D106.4 (DOUT): now also D105.2 (DIN); no longer D95.4 (DOUT)
- net at D45.2 (A): now also SW47.2; no longer SW47.1
- net at D63.2 (A): now also SW65.2; no longer SW65.1
- net at D71.2 (A): now also SW73.2; no longer SW73.1
- net RE 1: now reaches SW84.1
- net RE 1: now also A1.11 (GPIO8), SW15.S1, SW16.S1, SW83.1; no longer D82.2 (A)
- net at D25.2 (A): now also SW27.2; no longer SW26.1
- net at D3.2 (A): now also SW3.2; no longer SW3.1
- net at D47.2 (A): now also SW49.2; no longer SW49.1
- net at D9.2 (A): now also SW9.2; no longer SW9.1
- net at D31.2 (A): now also SW33.2; no longer SW33.1
- net at D21.2 (A): now also SW23.2; no longer SW22.1
- net at D103.2 (DIN): now also D104.4 (DOUT); no longer D102.4 (DOUT)
- net at D103.4 (DOUT): now also D102.2 (DIN); no longer D104.2 (DIN)
- net at D55.2 (A): now also SW57.2; no longer SW57.1
- net at D13.2 (A): now also SW13.2; no longer SW13.1
- net at D27.2 (A): now also SW29.2; no longer SW28.1
- net at D15.2 (A): now also SW17.2; no longer SW20.1
- net at D96.4 (DOUT): no longer D97.2 (DIN)
- net at D73.2 (A): now also SW75.2; no longer SW75.1
- net at D33.2 (A): now also SW35.2; no longer SW35.1
- net at D67.2 (A): now also SW69.2; no longer SW69.1
- net at D61.2 (A): now also SW63.2; no longer SW63.1
- net at D19.2 (A): now also SW21.2; no longer SW19.1
- net at D7.2 (A): now also SW7.2; no longer SW7.1
- net at D96.2 (DIN): now also D97.4 (DOUT)
- removed net COL 10: A1.24 (GPIO18), SW10.2, SW15.S1, SW16.S1
- removed net COL 6: A1.19 (GPIO14), SW26.2, SW30.2, SW36.2, SW45.2, SW54.2, SW6.2, SW63.2, SW72.2, SW81.2
- removed net COL 7: A1.20 (GPIO15), SW17.2, SW27.2, SW37.2, SW46.2, SW55.2, SW64.2, SW7.2, SW73.2, SW82.2
- removed net COL 8: A1.21 (GPIO16), SW18.2, SW28.2, SW38.2, SW47.2, SW56.2, SW65.2, SW74.2, SW8.2, SW83.2
- removed net COL 9: A1.22 (GPIO17), SW19.2, SW29.2, SW39.2, SW48.2, SW57.2, SW66.2, SW75.2, SW84.2, SW9.2
- removed net ROW 9: A1.11 (GPIO8), D74.1 (K), D75.1 (K), D76.1 (K), D77.1 (K), D78.1 (K), D79.1 (K), D80.1 (K), D81.1 (K), D82.1 (K)
- new net: D64.1 (K), SW66.2
- new net: D68.1 (K), SW70.2
- new net: D74.1 (K), SW76.2
- new net: D18.1 (K), SW20.2
- new net: D54.1 (K), SW56.2
- new net: D4.1 (K), SW4.2
- new net: D16.1 (K), SW18.2
- new net: D8.1 (K), SW8.2
- new net: D44.1 (K), SW46.2
- new net: D50.1 (K), SW52.2
- new net: D6.1 (K), SW6.2
- new net: D28.1 (K), SW30.2
- new net: D34.1 (K), SW36.2
- new net: D14.1 (K), SW14.2
- new net: D72.1 (K), SW74.2
- new net: D22.1 (K), SW24.2
- new net: D42.1 (K), SW44.2
- new net: D12.1 (K), SW12.2
- new net: D26.1 (K), SW28.2
- new net: D70.1 (K), SW72.2
- new net: D40.1 (K), SW42.2
- new net: D80.1 (K), SW82.2
- new net: D66.1 (K), SW68.2
- new net: D32.1 (K), SW34.2
- new net: D76.1 (K), SW78.2
- new net: D52.1 (K), SW54.2
- new net: D62.1 (K), SW64.2
- new net: D60.1 (K), SW62.2
- new net: D2.1 (K), SW2.2
- new net: D24.1 (K), SW26.2
- new net: D78.1 (K), SW80.2
- new net: D10.1 (K), SW10.2
- new net: D56.1 (K), SW58.2
- new net: D38.1 (K), SW40.2
- new net: D58.1 (K), SW60.2
- new net: D30.1 (K), SW32.2
- new net: D48.1 (K), SW50.2
- new net: D82.1 (K), SW84.2
- new net: D101.2 (DIN), D102.4 (DOUT)
- new net: D20.1 (K), SW22.2
- new net: D104.2 (DIN), D105.4 (DOUT)
- new net: D36.1 (K), SW38.2
- new net: D46.1 (K), SW48.2
- no-connect marks 0 -> 3
Other:
- note added: "DUPLEX MATRIX"
- note added: "STABILIZERS"
- note removed: "KEY MATRIX"
- moved on the sheet: D1, D10, D100, D101, D102, D103, D104, D105, D106, D2, D3, D4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
