File: Kicad_Nemo75/Kicad_Nemo75.kicad_pcb (KiCad board)
At the start: 2 copper layers, 340.5 x 144 mm, 0 parts

Commit message: doing pcb now first added correct step files to mx cherry hotswap and then editeed the its footprint to have hotswap on back layer, plus also started arranging stuff
Parts:
- added A1: RaspberryPi_Pico, Module:RaspberryPi_Pico_Common_Unspecified, F.Cu at (323.5, 378.4)
- added C1: C, Capacitor_SMD:C_1206_3216Metric_Pad1.33x1.80mm_HandSolder, F.Cu at (302.4, 367.5)
- added C2: C, Capacitor_SMD:C_1206_3216Metric_Pad1.33x1.80mm_HandSolder, F.Cu at (245.3, 366.7)
- added C3: C, Capacitor_SMD:C_1206_3216Metric_Pad1.33x1.80mm_HandSolder, F.Cu at (221.5, 366.7)
- added C4: C, Capacitor_SMD:C_1206_3216Metric_Pad1.33x1.80mm_HandSolder, F.Cu at (197.6, 366.7)
- added C5: C, Capacitor_SMD:C_1206_3216Metric_Pad1.33x1.80mm_HandSolder, F.Cu at (276.4, 368.6)
- added C6: C, Capacitor_SMD:C_1206_3216Metric_Pad1.33x1.80mm_HandSolder, F.Cu at (270.8, 368.6)
- added C7: C, Capacitor_SMD:C_1206_3216Metric_Pad1.33x1.80mm_HandSolder, F.Cu at (173.8, 366.7)
- added D1: D, Diode_THT:D_DO-35_SOD27_P7.62mm_Horizontal, B.Cu at (32.4, 391.7)
- added D10: D, Diode_THT:D_DO-35_SOD27_P7.62mm_Horizontal, B.Cu at (218.3, 391.7)
- added D100: SK6812, LED_SMD:LED_SK6812MINI-E_3.2x2.8mm_P1.5mm_ReverseMount, F.Cu at (197.9, 309.7)
- added D101: SK6812, LED_SMD:LED_SK6812MINI-E_3.2x2.8mm_P1.5mm_ReverseMount, F.Cu at (206.3, 275.6)
- added D102: SK6812, LED_SMD:LED_SK6812MINI-E_3.2x2.8mm_P1.5mm_ReverseMount, F.Cu at (206.3, 280.5)
- added D103: SK6812, LED_SMD:LED_SK6812MINI-E_3.2x2.8mm_P1.5mm_ReverseMount, F.Cu at (206.3, 285.4)
- added D104: SK6812, LED_SMD:LED_SK6812MINI-E_3.2x2.8mm_P1.5mm_ReverseMount, F.Cu at (206.3, 290.2)
- added D105: SK6812, LED_SMD:LED_SK6812MINI-E_3.2x2.8mm_P1.5mm_ReverseMount, F.Cu at (206.3, 295.1)
- added D106: SK6812, LED_SMD:LED_SK6812MINI-E_3.2x2.8mm_P1.5mm_ReverseMount, F.Cu at (206.3, 300.0)
- added D107: D, Diode_THT:D_DO-35_SOD27_P7.62mm_Horizontal, B.Cu at (306.4, 358.9)
- added D11: D, Diode_THT:D_DO-35_SOD27_P7.62mm_Horizontal, B.Cu at (237.2, 391.5)
- added D12: D, Diode_THT:D_DO-35_SOD27_P7.62mm_Horizontal, B.Cu at (256.5, 391.7)
- added D13: D, Diode_THT:D_DO-35_SOD27_P7.62mm_Horizontal, B.Cu at (275.4, 391.7)
- added D14: D, Diode_THT:D_DO-35_SOD27_P7.62mm_Horizontal, B.Cu at (299.2, 391.7)
- added D15: D, Diode_THT:D_DO-35_SOD27_P7.62mm_Horizontal, B.Cu at (32.4, 415.6)
- added D16: D, Diode_THT:D_DO-35_SOD27_P7.62mm_Horizontal, B.Cu at (51.4, 415.5)
- added D17: D, Diode_THT:D_DO-35_SOD27_P7.62mm_Horizontal, B.Cu at (70.5, 415.5)
- added D18: D, Diode_THT:D_DO-35_SOD27_P7.62mm_Horizontal, B.Cu at (89.5, 415.5)
- added D19: D, Diode_THT:D_DO-35_SOD27_P7.62mm_Horizontal, B.Cu at (108.6, 415.5)
- added D2: D, Diode_THT:D_DO-35_SOD27_P7.62mm_Horizontal, B.Cu at (56.2, 391.7)
- added D20: D, Diode_THT:D_DO-35_SOD27_P7.62mm_Horizontal, B.Cu at (127.9, 415.5)
- added D21: D, Diode_THT:D_DO-35_SOD27_P7.62mm_Horizontal, B.Cu at (146.7, 415.5)
- added D22: D, Diode_THT:D_DO-35_SOD27_P7.62mm_Horizontal, B.Cu at (165.8, 415.6)
- added D23: D, Diode_THT:D_DO-35_SOD27_P7.62mm_Horizontal, B.Cu at (184.8, 415.5)
- added D24: D, Diode_THT:D_DO-35_SOD27_P7.62mm_Horizontal, B.Cu at (203.8, 415.5)
- added D25: D, Diode_THT:D_DO-35_SOD27_P7.62mm_Horizontal, B.Cu at (222.9, 415.5)
- added D26: D, Diode_THT:D_DO-35_SOD27_P7.62mm_Horizontal, B.Cu at (241.9, 415.5)
- added D27: D, Diode_THT:D_DO-35_SOD27_P7.62mm_Horizontal, B.Cu at (261.1, 415.5)
- added D28: D, Diode_THT:D_DO-35_SOD27_P7.62mm_Horizontal, F.Cu at (197.6, 243.0)
- added D29: D, Diode_THT:D_DO-35_SOD27_P7.62mm_Horizontal, F.Cu at (197.6, 246.6)
- added D3: D, Diode_THT:D_DO-35_SOD27_P7.62mm_Horizontal, B.Cu at (75.2, 391.7)
- added D30: D, Diode_THT:D_DO-35_SOD27_P7.62mm_Horizontal, F.Cu at (197.6, 250.1)
- added D31: D, Diode_THT:D_DO-35_SOD27_P7.62mm_Horizontal, F.Cu at (197.6, 253.7)
- added D32: D, Diode_THT:D_DO-35_SOD27_P7.62mm_Horizontal, F.Cu at (197.6, 257.2)
- added D33: D, Diode_THT:D_DO-35_SOD27_P7.62mm_Horizontal, F.Cu at (197.6, 260.8)
- added D34: D, Diode_THT:D_DO-35_SOD27_P7.62mm_Horizontal, F.Cu at (197.6, 264.3)
- added D35: D, Diode_THT:D_DO-35_SOD27_P7.62mm_Horizontal, F.Cu at (197.6, 267.9)
- added D36: D, Diode_THT:D_DO-35_SOD27_P7.62mm_Horizontal, F.Cu at (197.6, 271.4)
- added D37: D, Diode_THT:D_DO-35_SOD27_P7.62mm_Horizontal, F.Cu at (208.4, 211.1)
- added D38: D, Diode_THT:D_DO-35_SOD27_P7.62mm_Horizontal, F.Cu at (208.4, 214.6)
- added D39: D, Diode_THT:D_DO-35_SOD27_P7.62mm_Horizontal, F.Cu at (208.4, 218.2)
- added D4: D, Diode_THT:D_DO-35_SOD27_P7.62mm_Horizontal, B.Cu at (94.4, 391.7)
- added D40: D, Diode_THT:D_DO-35_SOD27_P7.62mm_Horizontal, F.Cu at (208.4, 221.7)
- added D41: D, Diode_THT:D_DO-35_SOD27_P7.62mm_Horizontal, F.Cu at (208.4, 225.3)
- added D42: D, Diode_THT:D_DO-35_SOD27_P7.62mm_Horizontal, F.Cu at (208.4, 228.8)
- added D43: D, Diode_THT:D_DO-35_SOD27_P7.62mm_Horizontal, F.Cu at (208.4, 232.4)
- added D44: D, Diode_THT:D_DO-35_SOD27_P7.62mm_Horizontal, F.Cu at (208.4, 235.9)
- added D45: D, Diode_THT:D_DO-35_SOD27_P7.62mm_Horizontal, F.Cu at (208.4, 239.5)
- added D46: D, Diode_THT:D_DO-35_SOD27_P7.62mm_Horizontal, F.Cu at (208.4, 243.0)
- added D47: D, Diode_THT:D_DO-35_SOD27_P7.62mm_Horizontal, F.Cu at (208.4, 246.6)
- added D48: D, Diode_THT:D_DO-35_SOD27_P7.62mm_Horizontal, F.Cu at (208.4, 250.1)
- added D49: D, Diode_THT:D_DO-35_SOD27_P7.62mm_Horizontal, F.Cu at (208.4, 253.7)
- added D5: D, Diode_THT:D_DO-35_SOD27_P7.62mm_Horizontal, B.Cu at (113.3, 391.7)
- added D50: D, Diode_THT:D_DO-35_SOD27_P7.62mm_Horizontal, F.Cu at (208.4, 257.2)
- added D51: D, Diode_THT:D_DO-35_SOD27_P7.62mm_Horizontal, F.Cu at (208.4, 260.8)
- added D52: D, Diode_THT:D_DO-35_SOD27_P7.62mm_Horizontal, F.Cu at (208.4, 264.3)
- added D53: D, Diode_THT:D_DO-35_SOD27_P7.62mm_Horizontal, F.Cu at (208.4, 267.9)
- added D54: D, Diode_THT:D_DO-35_SOD27_P7.62mm_Horizontal, F.Cu at (208.4, 271.4)
- added D55: D, Diode_THT:D_DO-35_SOD27_P7.62mm_Horizontal, F.Cu at (219.2, 211.1)
- added D56: D, Diode_THT:D_DO-35_SOD27_P7.62mm_Horizontal, F.Cu at (219.2, 214.6)
- added D57: D, Diode_THT:D_DO-35_SOD27_P7.62mm_Horizontal, F.Cu at (219.2, 218.2)
- added D58: D, Diode_THT:D_DO-35_SOD27_P7.62mm_Horizontal, F.Cu at (219.2, 221.7)
- added D59: D, Diode_THT:D_DO-35_SOD27_P7.62mm_Horizontal, F.Cu at (219.2, 225.3)
- added D6: D, Diode_THT:D_DO-35_SOD27_P7.62mm_Horizontal, B.Cu at (137.2, 391.7)
- added D60: D, Diode_THT:D_DO-35_SOD27_P7.62mm_Horizontal, F.Cu at (219.2, 228.8)
- added D61: D, Diode_THT:D_DO-35_SOD27_P7.62mm_Horizontal, F.Cu at (219.2, 232.4)
- added D62: D, Diode_THT:D_DO-35_SOD27_P7.62mm_Horizontal, F.Cu at (219.2, 235.9)
- added D63: D, Diode_THT:D_DO-35_SOD27_P7.62mm_Horizontal, F.Cu at (219.2, 239.5)
- added D64: D, Diode_THT:D_DO-35_SOD27_P7.62mm_Horizontal, F.Cu at (219.2, 243.0)
- added D65: D, Diode_THT:D_DO-35_SOD27_P7.62mm_Horizontal, F.Cu at (219.2, 246.6)
- added D66: D, Diode_THT:D_DO-35_SOD27_P7.62mm_Horizontal, F.Cu at (219.2, 250.1)
- added D67: D, Diode_THT:D_DO-35_SOD27_P7.62mm_Horizontal, F.Cu at (219.2, 253.7)
- added D68: D, Diode_THT:D_DO-35_SOD27_P7.62mm_Horizontal, F.Cu at (219.2, 257.2)
- added D69: D, Diode_THT:D_DO-35_SOD27_P7.62mm_Horizontal, F.Cu at (219.2, 260.8)
- added D7: D, Diode_THT:D_DO-35_SOD27_P7.62mm_Horizontal, B.Cu at (156.2, 391.7)
- added D70: D, Diode_THT:D_DO-35_SOD27_P7.62mm_Horizontal, F.Cu at (219.2, 264.3)
- added D71: D, Diode_THT:D_DO-35_SOD27_P7.62mm_Horizontal, F.Cu at (219.2, 267.9)
- added D72: D, Diode_THT:D_DO-35_SOD27_P7.62mm_Horizontal, F.Cu at (219.2, 271.4)
- added D73: D, Diode_THT:D_DO-35_SOD27_P7.62mm_Horizontal, F.Cu at (230.0, 211.1)
- added D74: D, Diode_THT:D_DO-35_SOD27_P7.62mm_Horizontal, F.Cu at (230.0, 214.6)
- added D75: D, Diode_THT:D_DO-35_SOD27_P7.62mm_Horizontal, F.Cu at (230.0, 218.2)
- added D76: D, Diode_THT:D_DO-35_SOD27_P7.62mm_Horizontal, F.Cu at (230.0, 221.7)
- added D77: D, Diode_THT:D_DO-35_SOD27_P7.62mm_Horizontal, F.Cu at (230.0, 225.3)
- added D78: D, Diode_THT:D_DO-35_SOD27_P7.62mm_Horizontal, F.Cu at (230.0, 228.8)
- added D79: D, Diode_THT:D_DO-35_SOD27_P7.62mm_Horizontal, F.Cu at (230.0, 232.4)
- added D8: D, Diode_THT:D_DO-35_SOD27_P7.62mm_Horizontal, B.Cu at (175.3, 391.7)
- added D80: D, Diode_THT:D_DO-35_SOD27_P7.62mm_Horizontal, F.Cu at (230.0, 235.9)
- added D81: D, Diode_THT:D_DO-35_SOD27_P7.62mm_Horizontal, F.Cu at (230.0, 239.5)
- added D82: D, Diode_THT:D_DO-35_SOD27_P7.62mm_Horizontal, F.Cu at (230.0, 243.0)
- added D83: D, Diode_THT:D_DO-35_SOD27_P7.62mm_Horizontal, F.Cu at (230.0, 246.6)
- added D84: D, Diode_THT:D_DO-35_SOD27_P7.62mm_Horizontal, F.Cu at (230.0, 250.1)
- added D85: SK6812, LED_SMD:LED_SK6812MINI-E_3.2x2.8mm_P1.5mm_ReverseMount, F.Cu at (189.5, 275.6)
- added D86: SK6812, LED_SMD:LED_SK6812MINI-E_3.2x2.8mm_P1.5mm_ReverseMount, F.Cu at (189.5, 280.5)
- added D87: SK6812, LED_SMD:LED_SK6812MINI-E_3.2x2.8mm_P1.5mm_ReverseMount, F.Cu at (189.5, 285.4)
- added D88: SK6812, LED_SMD:LED_SK6812MINI-E_3.2x2.8mm_P1.5mm_ReverseMount, F.Cu at (189.5, 290.2)
- added D89: SK6812, LED_SMD:LED_SK6812MINI-E_3.2x2.8mm_P1.5mm_ReverseMount, F.Cu at (189.5, 295.1)
- added D9: D, Diode_THT:D_DO-35_SOD27_P7.62mm_Horizontal, B.Cu at (194.3, 391.7)
- added D90: SK6812, LED_SMD:LED_SK6812MINI-E_3.2x2.8mm_P1.5mm_ReverseMount, F.Cu at (189.5, 300.0)
- added D91: SK6812, LED_SMD:LED_SK6812MINI-E_3.2x2.8mm_P1.5mm_ReverseMount, F.Cu at (189.5, 304.8)
- added D92: SK6812, LED_SMD:LED_SK6812MINI-E_3.2x2.8mm_P1.5mm_ReverseMount, F.Cu at (189.5, 309.7)
- added D93: SK6812, LED_SMD:LED_SK6812MINI-E_3.2x2.8mm_P1.5mm_ReverseMount, F.Cu at (197.9, 275.6)
- added D94: SK6812, LED_SMD:LED_SK6812MINI-E_3.2x2.8mm_P1.5mm_ReverseMount, F.Cu at (197.9, 280.5)
- added D95: SK6812, LED_SMD:LED_SK6812MINI-E_3.2x2.8mm_P1.5mm_ReverseMount, F.Cu at (197.9, 285.4)
- added D96: SK6812, LED_SMD:LED_SK6812MINI-E_3.2x2.8mm_P1.5mm_ReverseMount, F.Cu at (197.9, 290.2)
- added D97: SK6812, LED_SMD:LED_SK6812MINI-E_3.2x2.8mm_P1.5mm_ReverseMount, F.Cu at (197.9, 295.1)
- added D98: SK6812, LED_SMD:LED_SK6812MINI-E_3.2x2.8mm_P1.5mm_ReverseMount, F.Cu at (197.9, 300.0)
- added D99: SK6812, LED_SMD:LED_SK6812MINI-E_3.2x2.8mm_P1.5mm_ReverseMount, F.Cu at (197.9, 304.8)
- added J1: Conn_01x08_Pin, Connector:Tag-Connect_TC2030-IDC-FP_2x03_P1.27mm_Vertical, F.Cu at (239.9, 289.9)
- added J2: USB_A, Connector_USB:USB_A_Molex_67643_Horizontal, F.Cu at (261.2, 366.2)
- added J4: USB_A, Connector_USB:USB_A_Molex_67643_Horizontal, F.Cu at (236.9, 366.2)
- added J5: USB_A, Connector_USB:USB_A_Molex_67643_Horizontal, F.Cu at (213.2, 366.2)
- added J6: USB_A, Connector_USB:USB_A_Molex_67643_Horizontal, F.Cu at (189.3, 366.3)
- added J7: USB_B_Micro, Connector_USB:USB_Micro-B_Wuerth_629105150521, F.Cu at (288.0, 357.1)
- added S1: MX_stab, PCM_marbastlib-mx:STAB_MX_P_6.25u, F.Cu at (100.6, 303.4)
- added S2: MX_stab, PCM_marbastlib-mx:STAB_MX_P_2.75u, F.Cu at (199.7, 137.8)
- added S3: MX_stab, PCM_marbastlib-mx:STAB_MX_P_2.75u, F.Cu at (199.7, 158.1)
- added S4: MX_stab, PCM_marbastlib-mx:STAB_MX_P_2u, F.Cu at (199.7, 178.3)
- added S5: MX_stab, PCM_marbastlib-mx:STAB_MX_P_2.25u, F.Cu at (199.7, 198.6)
- added SW1: SW_Push, PCM_marbastlib-mx:SW_MX_HS_CPG151101S11_1u, F.Cu at (28.6, 383.4)
- added SW10: SW_Push, PCM_marbastlib-mx:SW_MX_HS_CPG151101S11_1u, F.Cu at (214.3, 383.4)
- added SW11: SW_Push, PCM_marbastlib-mx:SW_MX_HS_CPG151101S11_1u, F.Cu at (233.4, 383.4)
- added SW12: SW_Push, PCM_marbastlib-mx:SW_MX_HS_CPG151101S11_1u, F.Cu at (252.4, 383.4)
- added SW13: SW_Push, PCM_marbastlib-mx:SW_MX_HS_CPG151101S11_1u, F.Cu at (271.5, 383.4)
- added SW14: SW_Push, PCM_marbastlib-mx:SW_MX_HS_CPG151101S11_1u, F.Cu at (295.3, 383.4)
- added SW15: RotaryEncoder_Switch, Rotary_Encoder:RotaryEncoder_Alps_EC11E-Switch_Vertical_H20mm, F.Cu at (212.6, 278.3)
- added SW16: RotaryEncoder_Switch, Rotary_Encoder:RotaryEncoder_Alps_EC11E-Switch_Vertical_H20mm, F.Cu at (212.6, 293.6)
- added SW17: SW_Push, PCM_marbastlib-mx:SW_MX_HS_CPG151101S11_1u, F.Cu at (28.6, 407.2)
- added SW18: SW_Push, PCM_marbastlib-mx:SW_MX_HS_CPG151101S11_1u, F.Cu at (47.6, 407.2)
- added SW19: SW_Push, PCM_marbastlib-mx:SW_MX_HS_CPG151101S11_1u, F.Cu at (66.6, 407.2)
- added SW2: SW_Push, PCM_marbastlib-mx:SW_MX_HS_CPG151101S11_1u, F.Cu at (52.4, 383.4)
- added SW20: SW_Push, PCM_marbastlib-mx:SW_MX_HS_CPG151101S11_1u, F.Cu at (85.7, 407.2)
- added SW21: SW_Push, PCM_marbastlib-mx:SW_MX_HS_CPG151101S11_1u, F.Cu at (104.8, 407.2)
- added SW22: SW_Push, PCM_marbastlib-mx:SW_MX_HS_CPG151101S11_1u, F.Cu at (123.8, 407.2)
- added SW23: SW_Push, PCM_marbastlib-mx:SW_MX_HS_CPG151101S11_1u, F.Cu at (142.9, 407.2)
- added SW24: SW_Push, PCM_marbastlib-mx:SW_MX_HS_CPG151101S11_1u, F.Cu at (161.9, 407.2)
- added SW25: SW_Push, PCM_marbastlib-mx:SW_MX_HS_CPG151101S11_1u, F.Cu at (181.0, 407.2)
- added SW26: SW_Push, PCM_marbastlib-mx:SW_MX_HS_CPG151101S11_1u, F.Cu at (200.0, 407.2)
- added SW27: SW_Push, PCM_marbastlib-mx:SW_MX_HS_CPG151101S11_1u, F.Cu at (219.1, 407.2)
- added SW28: SW_Push, PCM_marbastlib-mx:SW_MX_HS_CPG151101S11_1u, F.Cu at (238.1, 407.2)
- added SW29: SW_Push, PCM_marbastlib-mx:SW_MX_HS_CPG151101S11_1u, F.Cu at (257.2, 407.2)
- added SW3: SW_Push, PCM_marbastlib-mx:SW_MX_HS_CPG151101S11_1u, F.Cu at (71.4, 383.4)
- added SW30: SW_Push, PCM_marbastlib-mx:SW_MX_HS_CPG151101S11_1u, F.Cu at (90.3, 211.1)
- added SW31: SW_Push, PCM_marbastlib-mx:SW_MX_HS_CPG151101S11_1u, F.Cu at (90.3, 226.2)
- added SW32: SW_Push, PCM_marbastlib-mx:SW_MX_HS_CPG151101S11_1u, F.Cu at (90.3, 241.2)
- added SW33: SW_Push, PCM_marbastlib-mx:SW_MX_HS_CPG151101S11_1u, F.Cu at (90.3, 256.3)
- added SW34: SW_Push, PCM_marbastlib-mx:SW_MX_HS_CPG151101S11_1u, F.Cu at (90.3, 271.3)
- added SW35: SW_Push, PCM_marbastlib-mx:SW_MX_HS_CPG151101S11_1u, F.Cu at (90.3, 286.4)
- added SW36: SW_Push, PCM_marbastlib-mx:SW_MX_HS_CPG151101S11_1u, F.Cu at (107.5, 135.9)
- added SW37: SW_Push, PCM_marbastlib-mx:SW_MX_HS_CPG151101S11_1u, F.Cu at (107.5, 150.9)
- added SW38: SW_Push, PCM_marbastlib-mx:SW_MX_HS_CPG151101S11_1u, F.Cu at (107.5, 166.0)
- added SW39: SW_Push, PCM_marbastlib-mx:SW_MX_HS_CPG151101S11_1u, F.Cu at (107.5, 181.0)
- added SW4: SW_Push, PCM_marbastlib-mx:SW_MX_HS_CPG151101S11_1u, F.Cu at (90.5, 383.4)
- added SW40: SW_Push, PCM_marbastlib-mx:SW_MX_HS_CPG151101S11_1u, F.Cu at (107.5, 196.1)
- added SW41: SW_Push, PCM_marbastlib-mx:SW_MX_HS_CPG151101S11_1u, F.Cu at (107.5, 211.1)
- added SW42: SW_Push, PCM_marbastlib-mx:SW_MX_HS_CPG151101S11_1u, F.Cu at (107.5, 226.2)
- added SW43: SW_Push, PCM_marbastlib-mx:SW_MX_HS_CPG151101S11_1u, F.Cu at (107.5, 241.2)
- added SW44: SW_Push, PCM_marbastlib-mx:SW_MX_HS_CPG151101S11_1u, F.Cu at (107.5, 256.3)
- added SW45: SW_Push, PCM_marbastlib-mx:SW_MX_HS_CPG151101S11_1u, F.Cu at (107.5, 271.3)
- added SW46: SW_Push, PCM_marbastlib-mx:SW_MX_HS_CPG151101S11_1u, F.Cu at (107.5, 286.4)
- added SW47: SW_Push, PCM_marbastlib-mx:SW_MX_HS_CPG151101S11_1u, F.Cu at (124.6, 135.9)
- added SW48: SW_Push, PCM_marbastlib-mx:SW_MX_HS_CPG151101S11_1u, F.Cu at (124.6, 150.9)
- added SW49: SW_Push, PCM_marbastlib-mx:SW_MX_HS_CPG151101S11_1u, F.Cu at (124.6, 166.0)
- added SW5: SW_Push, PCM_marbastlib-mx:SW_MX_HS_CPG151101S11_1u, F.Cu at (109.5, 383.4)
- added SW50: SW_Push, PCM_marbastlib-mx:SW_MX_HS_CPG151101S11_1u, F.Cu at (124.6, 181.0)
- added SW51: SW_Push, PCM_marbastlib-mx:SW_MX_HS_CPG151101S11_1u, F.Cu at (124.6, 196.1)
- added SW52: SW_Push, PCM_marbastlib-mx:SW_MX_HS_CPG151101S11_1u, F.Cu at (124.6, 211.1)
- added SW53: SW_Push, PCM_marbastlib-mx:SW_MX_HS_CPG151101S11_1u, F.Cu at (124.6, 226.2)
- added SW54: SW_Push, PCM_marbastlib-mx:SW_MX_HS_CPG151101S11_1u, F.Cu at (124.6, 241.2)
- added SW55: SW_Push, PCM_marbastlib-mx:SW_MX_HS_CPG151101S11_1u, F.Cu at (124.6, 256.3)
- added SW56: SW_Push, PCM_marbastlib-mx:SW_MX_HS_CPG151101S11_1u, F.Cu at (124.6, 271.3)
- added SW57: SW_Push, PCM_marbastlib-mx:SW_MX_HS_CPG151101S11_1u, F.Cu at (124.6, 286.4)
- added SW58: SW_Push, PCM_marbastlib-mx:SW_MX_HS_CPG151101S11_1u, F.Cu at (141.8, 135.9)
- added SW59: SW_Push, PCM_marbastlib-mx:SW_MX_HS_CPG151101S11_1u, F.Cu at (141.8, 150.9)
- added SW6: SW_Push, PCM_marbastlib-mx:SW_MX_HS_CPG151101S11_1u, F.Cu at (133.3, 383.4)
- added SW60: SW_Push, PCM_marbastlib-mx:SW_MX_HS_CPG151101S11_1u, F.Cu at (141.8, 166.0)
- added SW61: SW_Push, PCM_marbastlib-mx:SW_MX_HS_CPG151101S11_1u, F.Cu at (141.8, 181.0)
- added SW62: SW_Push, PCM_marbastlib-mx:SW_MX_HS_CPG151101S11_1u, F.Cu at (141.8, 196.1)
- added SW63: SW_Push, PCM_marbastlib-mx:SW_MX_HS_CPG151101S11_1u, F.Cu at (141.8, 211.1)
- added SW64: SW_Push, PCM_marbastlib-mx:SW_MX_HS_CPG151101S11_1u, F.Cu at (141.8, 226.2)
- added SW65: SW_Push, PCM_marbastlib-mx:SW_MX_HS_CPG151101S11_1u, F.Cu at (141.8, 241.2)
- added SW66: SW_Push, PCM_marbastlib-mx:SW_MX_HS_CPG151101S11_1u, F.Cu at (141.8, 256.3)
- added SW67: SW_Push, PCM_marbastlib-mx:SW_MX_HS_CPG151101S11_1u, F.Cu at (141.8, 271.3)
- added SW68: SW_Push, PCM_marbastlib-mx:SW_MX_HS_CPG151101S11_1u, F.Cu at (141.8, 286.4)
- added SW69: SW_Push, PCM_marbastlib-mx:SW_MX_HS_CPG151101S11_1u, F.Cu at (158.9, 135.9)
- added SW7: SW_Push, PCM_marbastlib-mx:SW_MX_HS_CPG151101S11_1u, F.Cu at (152.4, 383.4)
- added SW70: SW_Push, PCM_marbastlib-mx:SW_MX_HS_CPG151101S11_1u, F.Cu at (158.9, 150.9)
- added SW71: SW_Push, PCM_marbastlib-mx:SW_MX_HS_CPG151101S11_1u, F.Cu at (158.9, 166.0)
- added SW72: SW_Push, PCM_marbastlib-mx:SW_MX_HS_CPG151101S11_1u, F.Cu at (158.9, 181.0)
- added SW73: SW_Push, PCM_marbastlib-mx:SW_MX_HS_CPG151101S11_1u, F.Cu at (158.9, 196.1)
- added SW74: SW_Push, PCM_marbastlib-mx:SW_MX_HS_CPG151101S11_1u, F.Cu at (158.9, 211.1)
- added SW75: SW_Push, PCM_marbastlib-mx:SW_MX_HS_CPG151101S11_1u, F.Cu at (158.9, 226.2)
- added SW76: SW_Push, PCM_marbastlib-mx:SW_MX_HS_CPG151101S11_1u, F.Cu at (158.9, 241.2)
- added SW77: SW_Push, PCM_marbastlib-mx:SW_MX_HS_CPG151101S11_1u, F.Cu at (158.9, 256.3)
- added SW78: SW_Push, PCM_marbastlib-mx:SW_MX_HS_CPG151101S11_1u, F.Cu at (158.9, 271.3)
- added SW79: SW_Push, PCM_marbastlib-mx:SW_MX_HS_CPG151101S11_1u, F.Cu at (158.9, 286.4)
- added SW8: SW_Push, PCM_marbastlib-mx:SW_MX_HS_CPG151101S11_1u, F.Cu at (171.4, 383.4)
- added SW80: SW_Push, PCM_marbastlib-mx:SW_MX_HS_CPG151101S11_1u, F.Cu at (176.1, 135.9)
- added SW81: SW_Push, PCM_marbastlib-mx:SW_MX_HS_CPG151101S11_1u, F.Cu at (176.1, 150.9)
- added SW82: SW_Push, PCM_marbastlib-mx:SW_MX_HS_CPG151101S11_1u, F.Cu at (176.1, 166.0)
- added SW83: SW_Push, PCM_marbastlib-mx:SW_MX_HS_CPG151101S11_1u, F.Cu at (176.1, 181.0)
- added SW84: SW_Push, PCM_marbastlib-mx:SW_MX_HS_CPG151101S11_1u, F.Cu at (176.1, 196.1)
- added SW9: SW_Push, PCM_marbastlib-mx:SW_MX_HS_CPG151101S11_1u, F.Cu at (190.5, 383.4)
- added U2: SL2.1A, Package_SO:SOIC-16_4.55x10.3mm_P1.27mm, B.Cu at (273.1, 361.1)
Other:
- outline, holes or cut-outs redrawn

Commit message: completed thw layout of the pcb added all the 3d models now js routing left
Parts:
- D100, D101, D102, D103, D104, D105, D106, D28, D29, D30, D31, D32, D33, D34, D35, D36, D37, D38, D39, D40, D41, D42, D43, D44, D45, D46, D47, D48, D49, D50, D51, D52, D53, D54, D55, D56, D57, D58, D59, D60, D61, D62, D63, D64, D65, D66, D67, D68, D69, D70, D71, D72, D73, D74, D75, D76, D77, D78, D79, D80, D81, D82, D83, D84, D85, D86, D87, D88, D89, D90, D91, D92, D93, D94, D95, D96, D97, D98, D99: moved to B.Cu
- J1: footprint Connector:Tag-Connect_TC2030-IDC-FP_2x03_P1.27mm_Vertical -> Connector_PinHeader_2.54mm:PinHeader_1x08_P2.54mm_Vertical
- S1: footprint PCM_marbastlib-mx:STAB_MX_P_6.25u -> PCM_marbastlib-mx:STAB_MX_6.25u
- S2: footprint PCM_marbastlib-mx:STAB_MX_P_2.75u -> PCM_marbastlib-mx:STAB_MX_2u
- S3: footprint PCM_marbastlib-mx:STAB_MX_P_2.75u -> PCM_marbastlib-mx:STAB_MX_2.75u
- S4: footprint PCM_marbastlib-mx:STAB_MX_P_2u -> PCM_marbastlib-mx:STAB_MX_2u
- S5: footprint PCM_marbastlib-mx:STAB_MX_P_2.25u -> PCM_marbastlib-mx:STAB_MX_2.25u
- SW31, SW44: footprint PCM_marbastlib-mx:SW_MX_HS_CPG151101S11_1u -> PCM_marbastlib-mx:SW_MX_HS_CPG151101S11_1.5u
- SW47: footprint PCM_marbastlib-mx:SW_MX_HS_CPG151101S11_1u -> PCM_marbastlib-mx:SW_MX_HS_CPG151101S11_1.75u
- SW75, SW76, SW77: footprint PCM_marbastlib-mx:SW_MX_HS_CPG151101S11_1u -> PCM_marbastlib-mx:SW_MX_HS_CPG151101S11_1.25u
- moved SW60 394.4 mm to (371.0, 487.0)
- moved SW61 371.1 mm to (351.9, 487.0)
- moved SW80 353.0 mm to (238.1, 483.4)
- moved S3 343.0 mm to (45.2, 464.3)
- moved SW81 342.2 mm to (257.2, 483.4)
- moved D73 341.8 mm to (34.8, 491.7), turned to 180 degrees
- moved SW82 341.5 mm to (292.6, 487.0)
- moved SW83 334.6 mm to (311.6, 487.0)
- moved SW69 330.5 mm to (195.3, 464.3)
- moved SW84 329.4 mm to (330.7, 487.0)
- moved SW45 328.7 mm to (370.9, 467.9)
- moved SW58 328.6 mm to (252.4, 445.3)
- moved SW59 326.6 mm to (283.4, 445.3)
- moved D74 325.8 mm to (58.6, 491.6), turned to 180 degrees
- moved SW47 321.9 mm to (35.7, 445.3)
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Connections:
- J1 pad 1: (no net) -> GND
- J1 pad 2: (no net) -> +3.3V
- J1 pad 3: (no net) -> SCL
- J1 pad 4: (no net) -> SDA
- J1 pad 5: (no net) -> RES
- J1 pad 6: (no net) -> DC
Other:
- board size 340.5 x 144 mm -> 364.3 x 144 mm

Commit message: pcb routing done tho it has too many vias so cool ;-;
Routing:
- net COL 1: track 0.00 -> 916.2 mm, vias 0 -> 13
- net COL 2: track 0.00 -> 817.3 mm, vias 0 -> 7
- net COL 4: track 0.00 -> 705.8 mm, vias 0 -> 10
- net COL 5: track 0.00 -> 656.3 mm, vias 0 -> 9
- net COL 3: track 0.00 -> 615.7 mm, vias 0 -> 4
- net ROW 1: track 0.00 -> 530.3 mm
- net ROW 5: track 0.00 -> 478.7 mm, vias 0 -> 3
- net ROW 8: track 0.00 -> 465.0 mm, vias 0 -> 3
- net ROW 6: track 0.00 -> 446.2 mm, vias 0 -> 7
- net ROW 3: track 0.00 -> 354.1 mm, vias 0 -> 4
- net ROW 2: track 0.00 -> 347.6 mm, vias 0 -> 2
- net ROW 4: track 0.00 -> 345.5 mm, vias 0 -> 4
- net ROW 7: track 0.00 -> 342.3 mm, vias 0 -> 2
- net RE 1: track 0.00 -> 264.0 mm, vias 0 -> 4
- net +3.3V: track 0.00 -> 254.1 mm, vias 0 -> 27
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- added copper zone on F.Cu, net +3.3V
- added copper zone on B.Cu, net GND
- added copper zone on B.Cu, net GND1
- added copper zone on F.Cu, net GND1
