File: Kicad_Nemo75/_restore_backup_2026-09-28T00-22-35-516/Kicad_Nemo75.kicad_sch (KiCad schematic)
At the start: 211 parts, among them J1 Conn_01x08_Pin, J2 USB_A, J4 USB_A, J5 USB_A, J6 USB_A, J7 USB_B_Micro, SW1 SW_Push, SW10 SW_Push, SW11 SW_Push, SW12 SW_Push, SW13 SW_Push, SW14 SW_Push, SW15 RotaryEncoder_Switch, SW16 RotaryEncoder_Switch, SW17 SW_Push, SW18 SW_Push, SW19 SW_Push, SW2 SW_Push, SW20 SW_Push, SW21 SW_Push, SW22 SW_Push, SW23 SW_Push, SW24 SW_Push, SW25 SW_Push, SW26 SW_Push, SW27 SW_Push, SW28 SW_Push, SW29 SW_Push, SW3 SW_Push, SW30 SW_Push, SW31 SW_Push, SW32 SW_Push, SW33 SW_Push, SW34 SW_Push, SW35 SW_Push, SW36 SW_Push, SW37 SW_Push, SW38 SW_Push, SW39 SW_Push, SW4 SW_Push, SW40 SW_Push, SW41 SW_Push, SW42 SW_Push, SW43 SW_Push, SW44 SW_Push, SW45 SW_Push, SW46 SW_Push, SW47 SW_Push, SW48 SW_Push, SW49 SW_Push, SW5 SW_Push, SW50 SW_Push, SW51 SW_Push, SW52 SW_Push, SW53 SW_Push, SW54 SW_Push, SW55 SW_Push, SW56 SW_Push, SW57 SW_Push, SW58 SW_Push, SW59 SW_Push, SW6 SW_Push, SW60 SW_Push, SW61 SW_Push, SW62 SW_Push, SW63 SW_Push, SW64 SW_Push, SW65 SW_Push, SW66 SW_Push, SW67 SW_Push, SW68 SW_Push, SW69 SW_Push, SW7 SW_Push, SW70 SW_Push, SW71 SW_Push, SW72 SW_Push, SW73 SW_Push, SW74 SW_Push, SW75 SW_Push, SW76 SW_Push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

Commit message: completed thw layout of the pcb added all the 3d models now js routing left
Parts:
- J1: footprint Connector_PinHeader_2.54mm:PinHeader_1x08_P2.54mm_Vertical -> Connector:Tag-Connect_TC2030-IDC-FP_2x03_P1.27mm_Vertical
- S4: footprint PCM_marbastlib-mx:STAB_MX_2u -> PCM_marbastlib-mx:STAB_MX_P_2u
- S5: footprint PCM_marbastlib-mx:STAB_MX_2.25u -> PCM_marbastlib-mx:STAB_MX_P_2.25u
Connections:
- net +3.3V: now also J1.VCC; no longer J1.2 (VCC)
- net BLK: now also J1.BLK; no longer J1.8 (BLK)
- net CS: now also J1.CS; no longer J1.7 (CS)
- net DC: now also J1.DC; no longer J1.6 (DC)
- net GND: now also J1.GND; no longer J1.1 (GND)
- net RES: now also J1.RES; no longer J1.5 (RES)
- net SCL: now also J1.SCL; no longer J1.3 (SCL)
- net SDA: now also J1.SDA; no longer J1.4 (SDA)
Changed lines of the file:
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@@
 			)
 		)
-		(property "Footprint" "Connector_PinHeader_2.54mm:PinHeader_1x08_P2.54mm_Vertical"
+		(property "Footprint" "Connector:Tag-Connect_TC2030-IDC-FP_2x03_P1.27mm_Vertical"
 			(at 261.62 62.23 0)
 			(hide yes)
@@
 			)
 		)
-		(pin "6"
+		(pin "VCC"
 		)
-		(pin "8"
+		(pin "RES"
 		)
-		(pin "7"
+		(pin "DC"
 		)
-		(pin "2"
+		(pin "SCL"
 		)
-		(pin "1"
+		(pin "SDA"
 		)
-		(pin "5"
+		(pin "CS"
 		)
-		(pin "3"
+		(pin "GND"
 		)
-		(pin "4"
+		(pin "BLK"
 		)
 		(instances
@@
 			)
 		)
-		(property "Footprint" "PCM_marbastlib-mx:STAB_MX_2u"
+		(property "Footprint" "PCM_marbastlib-mx:STAB_MX_P_2u"
 			(at 281.94 123.19 0)
 			(hide yes)
@@
 			)
 		)
-		(property "Footprint" "PCM_marbastlib-mx:STAB_MX_2.25u"
+		(property "Footprint" "PCM_marbastlib-mx:STAB_MX_P_2.25u"
 			(at 281.94 133.35 0)
 			(hide yes)
